File: RascalHat/RascalHat.sch (KiCad schematic (older format))
At the start: 13 parts, among them P1 Conn_01x06, U1 Conn_01x04, X1 Conn_01x02, X2 Conn_01x02

Commit message: update schematic
Parts:
- removed A1: Conn_01x08, symbol Connector_Generic:Conn_01x08
- removed J?: Conn_01x09, symbol Connector_Generic:Conn_01x09
- removed L2: Conn_01x07, symbol Connector_Generic:Conn_01x07
- removed P1: Conn_01x06, symbol Connector_Generic:Conn_01x06
- added A1: Conn_01x05, symbol Connector_Generic:Conn_01x05
- added C? (x4): CAP, symbol pspice:CAP
- added G1: Conn_01x04, symbol Connector_Generic:Conn_01x04
- added J? (x16): Conn_01x03, symbol Connector_Generic:Conn_01x03
- added L? (x2): INDUCTOR, symbol pspice:INDUCTOR
- added R? (x4): R, symbol Device:R
- added U?: MCP3008, symbol Analog_ADC:MCP3008
- added U?: PCA9685PW, Package_SO:TSSOP-28_4.4x9.7mm_P0.65mm, symbol Driver_LED:PCA9685PW
- added X3: Conn_01x02, symbol Connector_Generic:Conn_01x02
Connections:
- net labels added: +3V3, +5V, GND
- wire segments 0 -> 173
Other:
- moved on the sheet: B1, B2, E1, RR1, U1

Commit message: ...tweaking schematic....
Parts:
- removed B1: LM5166Y, Package_SON:Texas_S-PVSON-N10_ThermalVias, symbol Regulator_Switching:LM5166Y
- removed C? (x2): CAP, symbol pspice:CAP
- removed L?: INDUCTOR, symbol pspice:INDUCTOR
- removed R? (x2): R, symbol Device:R
- added PWR: Conn_01x02, symbol Connector_Generic:Conn_01x02
- added R? (x2): R, symbol Device:R
Connections:
- net +5V: now also PWR.1 (Pin_1)
- net GND: now also PWR.2 (Pin_2), R?.2
- net at R1.13 (GPIO27): now also R?.1, R?.1; no longer U1.3 (Pin_3)
- new net: R?.2, U1.3 (Pin_3)
Changed lines of the file:
@@
-$Comp
-L power:GND #PWR?
-U 1 1 6148974E
-P 8500 2000
-F 0 "#PWR?" H 8500 1750 50  0001 C CNN
-F 1 "GND" H 8505 1827 50  0000 C CNN
-F 2 "" H 8500 2000 50  0001 C CNN
-F 3 "" H 8500 2000 50  0001 C CNN
-	1    8500 2000
-	1    0    0    -1
-$EndComp
 $Comp
 L power:GND #PWR?
@@
 $EndComp
 $Comp
-L Regulator_Switching:LM5166Y B1
-U 1 1 613EF651
-P 8400 1500
-F 0 "B1" H 8400 2067 50  0000 C CNN
-F 1 "LM5166Y" H 8400 1976 50  0000 C CNN
-F 2 "Package_SON:Texas_S-PVSON-N10_ThermalVias" H 8450 1050 50  0001 L CNN
-F 3 "http://www.ti.com/lit/ds/symlink/lm5166.pdf" H 8400 2050 50  0001 C CNN
-	1    8400 1500
-	-1   0    0    -1
-$EndComp
-$Comp
-L power:+5V #PWR?
-U 1 1 614DAE78
-P 8000 1400
-F 0 "#PWR?" H 8000 1250 50  0001 C CNN
-F 1 "+5V" H 8015 1573 50  0000 C CNN
-F 2 "" H 8000 1400 50  0001 C CNN
-F 3 "" H 8000 1400 50  0001 C CNN
-	1    8000 1400
-	1    0    0    -1
-$EndComp
-$Comp
 L power:+3V3 #PWR?
 U 1 1 614DB584
@@
 $Comp
 L pspice:INDUCTOR L?
-U 1 1 614F1461
-P 7750 1200
-F 0 "L?" H 7750 1415 50  0000 C CNN
-F 1 "INDUCTOR" H 7750 1324 50  0000 C CNN
-F 2 "" H 7750 1200 50  0001 C CNN
-F 3 "~" H 7750 1200 50  0001 C CNN
-	1    7750 1200
-	1    0    0    -1
-$EndComp
-$Comp
-L pspice:INDUCTOR L?
 U 1 1 614F1B14
 P 7700 2750
@@
 F 3 "~" H 7700 2750 50  0001 C CNN
 	1    7700 2750
-	1    0    0    -1
-$EndComp
-$Comp
-L pspice:CAP C?
-U 1 1 614F3392
-P 9350 1450
-F 0 "C?" H 9528 1496 50  0000 L CNN
-F 1 "CAP" H 9528 1405 50  0000 L CNN
-F 2 "" H 9350 1450 50  0001 C CNN
-F 3 "~" H 9350 1450 50  0001 C CNN
-	1    9350 1450
-	1    0    0    -1
-$EndComp
-$Comp
-L power:GND #PWR?
-U 1 1 614F44CA
-P 9350 1700
-F 0 "#PWR?" H 9350 1450 50  0001 C CNN
-F 1 "GND" H 9355 1527 50  0000 C CNN
-F 2 "" H 9350 1700 50  0001 C CNN
-F 3 "" H 9350 1700 50  0001 C CNN
-	1    9350 1700
 	1    0    0    -1
 $EndComp
@@
 $Comp
 L Device:R R?
-U 1 1 61521CF6
-P 8950 1800
-F 0 "R?" V 8743 1800 50  0000 C CNN
-F 1 "R" V 8834 1800 50  0000 C CNN
-F 2 "" V 8880 1800 50  0001 C CNN
-F 3 "~" H 8950 1800 50  0001 C CNN
-	1    8950 1800
-	0    1    1    0
-$EndComp
-$Comp
-L Device:R R?
-U 1 1 61531CC6
-P 7500 1550
-F 0 "R?" H 7570 1596 50  0000 L CNN
-F 1 "R" H 7570 1505 50  0000 L CNN
-F 2 "" V 7430 1550 50  0001 C CNN
-F 3 "~" H 7500 1550 50  0001 C CNN
-	1    7500 1550
-	1    0    0    -1
-$EndComp
-$Comp
-L Device:R R?
 U 1 1 61532971
 P 7450 2600
@@
 $EndComp
 $Comp
-L pspice:CAP C?
-U 1 1 61537498
-P 7250 1700
-F 0 "C?" H 7428 1746 50  0000 L CNN
-F 1 "CAP" H 7428 1655 50  0000 L CNN
-F 2 "" H 7250 1700 50  0001 C CNN
-F 3 "~" H 7250 1700 50  0001 C CNN
-	1    7250 1700
-	0    -1   -1   0
-$EndComp
-$Comp
 L power:GND #PWR?
 U 1 1 6153A57A
@@
 	1    7450 1950
 	0    1    1    0
-$EndComp
-$Comp
-L power:GND #PWR?
-U 1 1 6153AB70
-P 7000 1700
-F 0 "#PWR?" H 7000 1450 50  0001 C CNN
-F 1 "GND" H 7005 1527 50  0000 C CNN
-F 2 "" H 7000 1700 50  0001 C CNN
-F 3 "" H 7000 1700 50  0001 C CNN
-	1    7000 1700
-	1    0    0    -1
 $EndComp
 $Comp
@@
 	3850 3250 4900 3250
 Wire Wire Line
-	1250 2850 3750 2850
-Wire Wire Line
-	3750 4450 4900 4450
-Wire Wire Line
 	7250 3950 7250 3250
 Wire Wire Line
@@
 	9550 600  9550 1200
 Wire Wire Line
-	9550 1200 9350 1200
-Wire Wire Line
 	10300 1050 9900 1050
 Wire Wire Line
@@
 	6550 1250 6300 1250
 Wire Wire Line
-	8800 1300 9200 1300
-Wire Wire Line
-	9200 1300 9200 1200
-Connection ~ 9200 1200
-Wire Wire Line
-	9200 1200 8800 1200
-Wire Wire Line
 	8750 2850 9200 2850
 Wire Wire Line
@@
 Wire Wire Line
 	9200 2750 9350 2750
-Connection ~ 9350 1200
-Wire Wire Line
-	9350 1200 9200 1200
 Connection ~ 9350 2750
 Wire Wire Line
@@
 Connection ~ 7950 2950
 Wire Wire Line
-	8000 1400 7500 1400
-Wire Wire Line
-	7500 1400 7500 1200
-Connection ~ 8000 1400
-Wire Wire Line
 	9050 3150 9050 3350
 Connection ~ 8450 3550
@@
 Wire Wire Line
 	8700 3550 8450 3550
-Wire Wire Line
-	8000 1700 8000 2250
-Wire Wire Line
-	8000 2250 8700 2250
-Wire Wire Line
-	8700 2000 8500 2000
-Wire Wire Line
-	8700 2000 8700 2250
-Connection ~ 8500 2000
-Connection ~ 8700 2000
 Connection ~ 9050 3350
 Wire Wire Line
@@
 Wire Wire Line
 	8750 3150 9050 3150
-Wire Wire Line
-	8800 1600 9100 1600
-Wire Wire Line
-	8700 2000 9100 2000
-Wire Wire Line
-	9100 1600 9100 1800
-Connection ~ 9100 1800
-Wire Wire Line
-	9100 1800 9100 2000
-Connection ~ 7500 1400
 Wire Wire Line
 	3750 2850 3750 4450
@@
 	1    0    0    -1
 $EndComp
+$Comp
+L Connector_Generic:Conn_01x02 PWR
+U 1 1 615C23C6
+P 10500 2250
+F 0 "PWR" H 10580 2242 50  0000 L CNN
+F 1 "Conn_01x02" H 10580 2151 50  0000 L CNN
+F 2 "" H 10500 2250 50  0001 C CNN
+F 3 "~" H 10500 2250 50  0001 C CNN
+	1    10500 2250
+	1    0    0    -1
+$EndComp
+$Comp
+L power:GND #PWR?
+U 1 1 615C2CAF
+P 10300 2350
+F 0 "#PWR?" H 10300 2100 50  0001 C CNN
+F 1 "GND" H 10305 2177 50  0000 C CNN
+F 2 "" H 10300 2350 50  0001 C CNN
+F 3 "" H 10300 2350 50  0001 C CNN
+	1    10300 2350
+	1    0    0    -1
+$EndComp
+$Comp
+L power:+5V #PWR?
+U 1 1 615D497E
+P 10300 2250
+F 0 "#PWR?" H 10300 2100 50  0001 C CNN
+F 1 "+5V" H 10315 2423 50  0000 C CNN
+F 2 "" H 10300 2250 50  0001 C CNN
+F 3 "" H 10300 2250 50  0001 C CNN
+	1    10300 2250
+	1    0    0    -1
+$EndComp
+$Comp
+L power:GND #PWR?
+U 1 1 616F5E45
+P 3000 4450
+F 0 "#PWR?" H 3000 4200 50  0001 C CNN
+F 1 "GND" H 3005 4277 50  0000 C CNN
+F 2 "" H 3000 4450 50  0001 C CNN
+F 3 "" H 3000 4450 50  0001 C CNN
+	1    3000 4450
+	1    0    0    -1
+$EndComp
+$Comp
+L Device:R R?
+U 1 1 616F82EF
+P 3350 4450
+F 0 "R?" V 3143 4450 50  0000 C CNN
+F 1 "R" V 3234 4450 50  0000 C CNN
+F 2 "" V 3280 4450 50  0001 C CNN
+F 3 "~" H 3350 4450 50  0001 C CNN
+	1    3350 4450
+	0    1    1    0
+$EndComp
+$Comp
+L Device:R R?
+U 1 1 616F8D77
+P 2350 2850
+F 0 "R?" V 2143 2850 50  0000 C CNN
+F 1 "R" V 2234 2850 50  0000 C CNN
+F 2 "" V 2280 2850 50  0001 C CNN
+F 3 "~" H 2350 2850 50  0001 C CNN
+	1    2350 2850
+	0    1    1    0
+$EndComp
+Wire Wire Line
+	2500 2850 3750 2850
+Wire Wire Line
+	2200 2850 1250 2850
+Wire Wire Line
+	3750 4450 3500 4450
+Wire Wire Line
+	3200 4450 3000 4450
+Wire Wire Line
+	3750 4450 4900 4450
+Connection ~ 3750 4450
 $EndSCHEMATC

Commit message: everything except accelerometer done
Parts:
- added L2: Conn_01x07, symbol Connector_Generic:Conn_01x07
- added U?: MPU-6050, Sensor_Motion:InvenSense_QFN-24_4x4mm_P0.5mm, symbol Sensor_Motion:MPU-6050
Connections:
- wire segments 161 -> 173
Changed lines of the file:
@@
 	5100 1800 5100 1750
 Wire Wire Line
-	850  1350 700  1350
-Wire Wire Line
-	700  1350 700  1750
-Wire Wire Line
-	700  1750 5000 1750
-Wire Wire Line
-	5000 1750 5000 1650
-Wire Wire Line
-	5000 1650 5100 1650
-Wire Wire Line
 	850  1550 5100 1550
 Wire Wire Line
@@
 Wire Wire Line
 	6850 4450 6500 4450
-Wire Wire Line
-	6850 5650 6850 4450
 Connection ~ 7250 3950
 Connection ~ 7050 4050
@@
 	4600 2850 4900 2850
 Wire Wire Line
-	7250 3950 7250 5850
-Wire Wire Line
-	7050 4050 7050 5950
+	7250 3950 7250 5050
 Wire Wire Line
 	850  4700 4400 4700
@@
 	3750 4450 4900 4450
 Connection ~ 3750 4450
+$Comp
+L Connector_Generic:Conn_01x07 L2
+U 1 1 61754839
+P 1800 1050
+F 0 "L2" H 1880 1092 50  0000 L CNN
+F 1 "Conn_01x07" H 1880 1001 50  0000 L CNN
+F 2 "" H 1800 1050 50  0001 C CNN
+F 3 "~" H 1800 1050 50  0001 C CNN
+	1    1800 1050
+	-1   0    0    1
+$EndComp
+$Comp
+L Sensor_Motion:MPU-6050 U?
+U 1 1 6175D5AD
+P 8700 5250
+F 0 "U?" H 8700 4461 50  0000 C CNN
+F 1 "MPU-6050" H 8700 4370 50  0000 C CNN
+F 2 "Sensor_Motion:InvenSense_QFN-24_4x4mm_P0.5mm" H 8700 4450 50  0001 C CNN
+F 3 "https://store.invensense.com/datasheets/invensense/MPU-6050_DataSheet_V3%204.pdf" H 8700 5100 50  0001 C CNN
+	1    8700 5250
+	1    0    0    -1
+$EndComp
+$Comp
+L power:GND #PWR?
+U 1 1 617691CA
+P 2000 1250
+F 0 "#PWR?" H 2000 1000 50  0001 C CNN
+F 1 "GND" V 2005 1122 50  0000 R CNN
+F 2 "" H 2000 1250 50  0001 C CNN
+F 3 "" H 2000 1250 50  0001 C CNN
+	1    2000 1250
+	0    -1   -1   0
+$EndComp
+$Comp
+L power:+5V #PWR?
+U 1 1 6176A224
+P 2000 1350
+F 0 "#PWR?" H 2000 1200 50  0001 C CNN
+F 1 "+5V" V 2015 1478 50  0000 L CNN
+F 2 "" H 2000 1350 50  0001 C CNN
+F 3 "" H 2000 1350 50  0001 C CNN
+	1    2000 1350
+	0    1    1    0
+$EndComp
+Wire Wire Line
+	2000 1150 2650 1150
+Wire Wire Line
+	2650 1150 2650 1700
+Wire Wire Line
+	2650 1700 5100 1700
+Wire Wire Line
+	5100 1700 5100 1650
+Wire Wire Line
+	2000 1050 2800 1050
+Wire Wire Line
+	2800 1050 2800 1350
+Wire Wire Line
+	2800 1350 5100 1350
+Wire Wire Line
+	2000 850  3000 850
+Wire Wire Line
+	3000 850  3000 1250
+Wire Wire Line
+	3000 1250 5100 1250
+Wire Wire Line
+	2000 750  3450 750
+Wire Wire Line
+	3450 750  3450 1150
+Wire Wire Line
+	3450 1150 5100 1150
+Wire Wire Line
+	6850 5650 6850 4450
+Wire Wire Line
+	8000 4950 7050 4950
+Wire Wire Line
+	7050 4050 7050 4950
+Connection ~ 7050 4950
+Wire Wire Line
+	7050 4950 7050 5950
+Wire Wire Line
+	8000 5050 7250 5050
+Connection ~ 7250 5050
+Wire Wire Line
+	7250 5050 7250 5850
 $EndSCHEMATC

Commit message: using only connector for accelerometer
Parts:
- removed U?: MPU-6050, Sensor_Motion:InvenSense_QFN-24_4x4mm_P0.5mm, symbol Sensor_Motion:MPU-6050
Connections:
- wire segments 173 -> 169
Changed lines of the file:
@@
 	4600 2850 4900 2850
-Wire Wire Line
-	7250 3950 7250 5050
 Wire Wire Line
 	850  4700 4400 4700
@@
 $EndComp
 $Comp
-L Sensor_Motion:MPU-6050 U?
-U 1 1 6175D5AD
-P 8700 5250
-F 0 "U?" H 8700 4461 50  0000 C CNN
-F 1 "MPU-6050" H 8700 4370 50  0000 C CNN
-F 2 "Sensor_Motion:InvenSense_QFN-24_4x4mm_P0.5mm" H 8700 4450 50  0001 C CNN
-F 3 "https://store.invensense.com/datasheets/invensense/MPU-6050_DataSheet_V3%204.pdf" H 8700 5100 50  0001 C CNN
-	1    8700 5250
-	1    0    0    -1
-$EndComp
-$Comp
 L power:GND #PWR?
 U 1 1 617691CA
@@
 	6850 5650 6850 4450
 Wire Wire Line
-	8000 4950 7050 4950
-Wire Wire Line
-	7050 4050 7050 4950
-Connection ~ 7050 4950
-Wire Wire Line
-	7050 4950 7050 5950
-Wire Wire Line
-	8000 5050 7250 5050
-Connection ~ 7250 5050
-Wire Wire Line
-	7250 5050 7250 5850
+	7050 4050 7050 5950
+Wire Wire Line
+	7250 3950 7250 5850
 $EndSCHEMATC

Commit message: added extra adc
Parts:
- removed L2: Conn_01x07, symbol Connector_Generic:Conn_01x07
- added L?: Conn_01x07, symbol Connector_Generic:Conn_01x07
- added U?: MCP3008, symbol Analog_ADC:MCP3008
Connections:
- net +3V3: now also U?.15 (Vref), U?.16 (Vdd)
- net +5V: now also L?.1 (Pin_1)
- net GND: now also L?.2 (Pin_2), U?.14 (AGND), U?.9 (DGND)
- net at R1.19 (MOSI0/GPIO10), U?.11 (Din): now also U?.11 (Din)
- net at R1.21 (MISO0/GPIO9), U?.12 (Dout): now also U?.12 (Dout)
- net at R1.23 (SCLK0/GPIO11), U?.13 (CLK): now also U?.13 (CLK)
- net at R1.26 (~CE1~/GPIO7): now also U?.10 (~CS~/SHDN)
- net at L1.5 (Pin_5): now also U?.7 (CH6)
- new net: L?.3 (Pin_3), U?.4 (CH3)
- new net: L?.4 (Pin_4), U?.5 (CH4)
- new net: L?.5 (Pin_5), U?.6 (CH5)
- new net: L?.6 (Pin_6), U?.7 (CH6)
- new net: L?.7 (Pin_7), U?.8 (CH7)
Other:
- note added: "Divide 5V output to get 3.3V"
Changed lines of the file:
@@
 	6850 1450 6850 4150
 Wire Wire Line
-	6850 4150 6500 4150
+	6850 4150 6750 4150
 Wire Wire Line
 	6500 4250 6550 4250
@@
 	3750 4450 4900 4450
 Connection ~ 3750 4450
-$Comp
-L Connector_Generic:Conn_01x07 L2
-U 1 1 61754839
-P 1800 1050
-F 0 "L2" H 1880 1092 50  0000 L CNN
-F 1 "Conn_01x07" H 1880 1001 50  0000 L CNN
-F 2 "" H 1800 1050 50  0001 C CNN
-F 3 "~" H 1800 1050 50  0001 C CNN
-	1    1800 1050
-	-1   0    0    1
-$EndComp
-$Comp
-L power:GND #PWR?
-U 1 1 617691CA
-P 2000 1250
-F 0 "#PWR?" H 2000 1000 50  0001 C CNN
-F 1 "GND" V 2005 1122 50  0000 R CNN
-F 2 "" H 2000 1250 50  0001 C CNN
-F 3 "" H 2000 1250 50  0001 C CNN
-	1    2000 1250
+Wire Wire Line
+	5100 1700 5100 1650
+Wire Wire Line
+	6850 5650 6850 4450
+Wire Wire Line
+	7050 4050 7050 5950
+Wire Wire Line
+	7250 3950 7250 5850
+Text Notes 2600 2950 0    50   ~ 0
+Divide 5V output to get 3.3V
+$Comp
+L Analog_ADC:MCP3008 U?
+U 1 1 6174A612
+P 8150 5250
+F 0 "U?" H 8150 5931 50  0000 C CNN
+F 1 "MCP3008" H 8150 5840 50  0000 C CNN
+F 2 "" H 8250 5350 50  0001 C CNN
+F 3 "http://ww1.microchip.com/downloads/en/DeviceDoc/21295d.pdf" H 8250 5350 50  0001 C CNN
+	1    8150 5250
+	-1   0    0    -1
+$EndComp
+$Comp
+L power:+3V3 #PWR?
+U 1 1 6174A618
+P 7950 4750
+F 0 "#PWR?" H 7950 4600 50  0001 C CNN
+F 1 "+3V3" H 7965 4923 50  0000 C CNN
+F 2 "" H 7950 4750 50  0001 C CNN
+F 3 "" H 7950 4750 50  0001 C CNN
+	1    7950 4750
+	-1   0    0    -1
+$EndComp
+$Comp
+L power:+3V3 #PWR?
+U 1 1 6174A61E
+P 8250 4750
+F 0 "#PWR?" H 8250 4600 50  0001 C CNN
+F 1 "+3V3" H 8265 4923 50  0000 C CNN
+F 2 "" H 8250 4750 50  0001 C CNN
+F 3 "" H 8250 4750 50  0001 C CNN
+	1    8250 4750
+	-1   0    0    -1
+$EndComp
+$Comp
+L power:GND #PWR?
+U 1 1 6174A624
+P 7950 5850
+F 0 "#PWR?" H 7950 5600 50  0001 C CNN
+F 1 "GND" H 7955 5677 50  0000 C CNN
+F 2 "" H 7950 5850 50  0001 C CNN
+F 3 "" H 7950 5850 50  0001 C CNN
+	1    7950 5850
+	-1   0    0    -1
+$EndComp
+$Comp
+L power:GND #PWR?
+U 1 1 6174A62A
+P 8250 5850
+F 0 "#PWR?" H 8250 5600 50  0001 C CNN
+F 1 "GND" H 8255 5677 50  0000 C CNN
+F 2 "" H 8250 5850 50  0001 C CNN
+F 3 "" H 8250 5850 50  0001 C CNN
+	1    8250 5850
+	-1   0    0    -1
+$EndComp
+$Comp
+L Connector_Generic:Conn_01x07 L?
+U 1 1 6175D0D5
+P 10850 5350
+F 0 "L?" H 10930 5392 50  0000 L CNN
+F 1 "Conn_01x07" H 10930 5301 50  0000 L CNN
+F 2 "" H 10850 5350 50  0001 C CNN
+F 3 "~" H 10850 5350 50  0001 C CNN
+	1    10850 5350
+	1    0    0    -1
+$EndComp
+$Comp
+L power:GND #PWR?
+U 1 1 6175D0DB
+P 10650 5150
+F 0 "#PWR?" H 10650 4900 50  0001 C CNN
+F 1 "GND" V 10655 5022 50  0000 R CNN
+F 2 "" H 10650 5150 50  0001 C CNN
+F 3 "" H 10650 5150 50  0001 C CNN
+	1    10650 5150
+	0    1    1    0
+$EndComp
+$Comp
+L power:+5V #PWR?
+U 1 1 6175D0E1
+P 10650 5050
+F 0 "#PWR?" H 10650 4900 50  0001 C CNN
+F 1 "+5V" V 10665 5178 50  0000 L CNN
+F 2 "" H 10650 5050 50  0001 C CNN
+F 3 "" H 10650 5050 50  0001 C CNN
+	1    10650 5050
 	0    -1   -1   0
 $EndComp
-$Comp
-L power:+5V #PWR?
-U 1 1 6176A224
-P 2000 1350
-F 0 "#PWR?" H 2000 1200 50  0001 C CNN
-F 1 "+5V" V 2015 1478 50  0000 L CNN
-F 2 "" H 2000 1350 50  0001 C CNN
-F 3 "" H 2000 1350 50  0001 C CNN
-	1    2000 1350
-	0    1    1    0
-$EndComp
-Wire Wire Line
-	2000 1150 2650 1150
-Wire Wire Line
-	2650 1150 2650 1700
-Wire Wire Line
-	2650 1700 5100 1700
-Wire Wire Line
-	5100 1700 5100 1650
-Wire Wire Line
-	2000 1050 2800 1050
-Wire Wire Line
-	2800 1050 2800 1350
-Wire Wire Line
-	2800 1350 5100 1350
-Wire Wire Line
-	2000 850  3000 850
-Wire Wire Line
-	3000 850  3000 1250
-Wire Wire Line
-	3000 1250 5100 1250
-Wire Wire Line
-	2000 750  3450 750
-Wire Wire Line
-	3450 750  3450 1150
-Wire Wire Line
-	3450 1150 5100 1150
-Wire Wire Line
-	6850 5650 6850 4450
-Wire Wire Line
-	7050 4050 7050 5950
-Wire Wire Line
-	7250 3950 7250 5850
+Wire Wire Line
+	8750 5250 10650 5250
+Wire Wire Line
+	8750 5350 10650 5350
+Wire Wire Line
+	10650 5450 8750 5450
+Wire Wire Line
+	8750 5550 10650 5550
+Wire Wire Line
+	8750 5650 10650 5650
+Wire Wire Line
+	7550 5150 6550 5150
+Wire Wire Line
+	6550 5150 6550 4250
+Connection ~ 6550 4250
+Wire Wire Line
+	7550 5250 6650 5250
+Wire Wire Line
+	6650 5250 6650 4050
+Connection ~ 6650 4050
+Wire Wire Line
+	7550 5350 6750 5350
+Wire Wire Line
+	6750 5350 6750 4150
+Connection ~ 6750 4150
+Wire Wire Line
+	6750 4150 6500 4150
+Wire Wire Line
+	7550 5450 6950 5450
+Wire Wire Line
+	6950 5450 6950 3850
+Wire Wire Line
+	6950 3850 6500 3850
+Wire Wire Line
+	850  1350 750  1350
+Wire Wire Line
+	750  1350 750  1700
+Wire Wire Line
+	750  1700 5100 1700
 $EndSCHEMATC
