File: RascalHat/AS5600 Magnetic Encoder.sch (KiCad schematic (older format))
At the start: 3 parts, among them J18 Conn_01x07_Male, J19 Conn_01x03_Male, J20 Conn_01x03_Male

Commit message: schematic done, symbol-footprint done, pcb started
Parts:
- J18: footprint (none) -> Connector_JST:JST_EH_B7B-EH-A_1x07_P2.50mm_Vertical
- J19, J20: footprint (none) -> Connector_JST:JST_EH_B3B-EH-A_1x03_P2.50mm_Vertical
Changed lines of the file:
@@
 $Descr A4 11693 8268
 encoding utf-8
-Sheet 6 6
+Sheet 8 8
 Title ""
 Date ""
@@
 F 0 "J18" H 5022 3732 50  0000 R CNN
 F 1 "Conn_01x07_Male" H 5022 3823 50  0000 R CNN
-F 2 "" H 5050 3800 50  0001 C CNN
+F 2 "Connector_JST:JST_EH_B7B-EH-A_1x07_P2.50mm_Vertical" H 5050 3800 50  0001 C CNN
 F 3 "~" H 5050 3800 50  0001 C CNN
 	1    5050 3800
@@
 F 0 "J19" H 6372 3682 50  0000 R CNN
 F 1 "Conn_01x03_Male" H 6372 3773 50  0000 R CNN
-F 2 "" H 6400 3750 50  0001 C CNN
+F 2 "Connector_JST:JST_EH_B3B-EH-A_1x03_P2.50mm_Vertical" H 6400 3750 50  0001 C CNN
 F 3 "~" H 6400 3750 50  0001 C CNN
 	1    6400 3750
@@
 F 0 "J20" H 6372 4332 50  0000 R CNN
 F 1 "Conn_01x03_Male" H 6372 4423 50  0000 R CNN
-F 2 "" H 6400 4400 50  0001 C CNN
+F 2 "Connector_JST:JST_EH_B3B-EH-A_1x03_P2.50mm_Vertical" H 6400 4400 50  0001 C CNN
 F 3 "~" H 6400 4400 50  0001 C CNN
 	1    6400 4400
