File: RascalHat/Accelerometer MPU6050.sch (KiCad schematic (older format))
At the start: 1 part, among them J1 Conn_01x08_Male

Commit message: schematic done, symbol-footprint done, pcb started
Parts:
- J1: footprint (none) -> Connector_JST:JST_EH_B8B-EH-A_1x08_P2.50mm_Vertical
Changed lines of the file:
@@
 $Descr A4 11693 8268
 encoding utf-8
-Sheet 3 6
+Sheet 3 8
 Title ""
 Date ""
@@
 F 0 "J1" H 5472 3474 50  0000 R CNN
 F 1 "Conn_01x08_Male" H 5472 3383 50  0000 R CNN
-F 2 "" H 5500 3500 50  0001 C CNN
+F 2 "Connector_JST:JST_EH_B8B-EH-A_1x08_P2.50mm_Vertical" H 5500 3500 50  0001 C CNN
 F 3 "~" H 5500 3500 50  0001 C CNN
 	1    5500 3500

Commit message: schematic updated, all footprints created, pcb layout started
Parts:
- J1: footprint Connector_JST:JST_EH_B8B-EH-A_1x08_P2.50mm_Vertical -> RascalHat:MPU-6050-Module
Changed lines of the file:
@@
 F 0 "J1" H 5472 3474 50  0000 R CNN
 F 1 "Conn_01x08_Male" H 5472 3383 50  0000 R CNN
-F 2 "Connector_JST:JST_EH_B8B-EH-A_1x08_P2.50mm_Vertical" H 5500 3500 50  0001 C CNN
+F 2 "RascalHat:MPU-6050-Module" H 5500 3500 50  0001 C CNN
 F 3 "~" H 5500 3500 50  0001 C CNN
 	1    5500 3500
