File: RascalHat/RascalHat.kicad_pcb (KiCad board)
At the start: 2 copper layers, 65 x 56 mm, 39 parts, among them J1 Conn_01x08_Male, J10 Conn_01x04_Male, J11 Conn_01x03_Male, J12 Conn_01x03_Male, J13 Conn_01x07_Male, J14 Conn_01x07_Male, J15 Conn_01x07_Male, J16 Conn_01x06_Male, J17 Conn_01x02_Male, J18 Conn_01x07_Male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

Commit message: schematic updated, all footprints created, pcb layout started
Parts:
- removed J3: Conn_01x04_Male, Connector_JST:JST_EH_B4B-EH-A_1x04_P2.50mm_Vertical
- added C5: CP1, Capacitor_SMD:CP_Elec_4x4.5, F.Cu at (8.51, 15.6)
- added C6: 0.1uF, Capacitor_SMD:C_0805_2012Metric, F.Cu at (91.4, -1.95)
- added D2: LED, Diode_SMD:D_0805_2012Metric, F.Cu at (101.9, -0.51)
- added D3: LED, Diode_SMD:D_0805_2012Metric, F.Cu at (114.2, -1.91)
- added D4: LED, Diode_SMD:D_0805_2012Metric, F.Cu at (106.4, -0.51)
- added R10: 3k3, Resistor_SMD:R_0805_2012Metric, F.Cu at (115.2, 1.09)
- added R8: 470, Resistor_SMD:R_0805_2012Metric, F.Cu at (110.8, 1.09)
- added R9: 2k2, Resistor_SMD:R_0805_2012Metric, F.Cu at (118.6, -1.95)
- added U1: MCP3008-I_P, Package_SO:SOIC-16_3.9x9.9mm_P1.27mm, B.Cu at (60.7, 44.1)
- added U2: MCP3008-I_P, Package_SO:SOIC-16_3.9x9.9mm_P1.27mm, B.Cu at (60.7, 33.4)
- added U5: TXB0108PWR, Package_SO:TSSOP-20_4.4x6.5mm_P0.65mm, F.Cu at (12.8, 32.3)
- J1: footprint Connector_JST:JST_EH_B8B-EH-A_1x08_P2.50mm_Vertical -> RascalHat:MPU-6050-Module
- J2: footprint Connector_JST:JST_EH_B9B-EH-A_1x09_P2.50mm_Vertical -> RascalHat:SIM808-Module
- J4: value Conn_01x08_Male -> Conn_01x04_Male; footprint Connector_JST:JST_EH_B8B-EH-A_1x08_P2.50mm_Vertical -> Connector_JST:JST_EH_B4B-EH-A_1x04_P2.50mm_Vertical
- J5: value Conn_01x08_Male -> Conn_01x07_Male; footprint Connector_JST:JST_EH_B8B-EH-A_1x08_P2.50mm_Vertical -> Connector_JST:JST_EH_B7B-EH-A_1x07_P2.50mm_Vertical
- J6: footprint Connector_AMASS:AMASS_XT30U-M_1x02_P5.0mm_Vertical -> RascalHat:XT30U-M-Horizontal
- J7: footprint Connector_AMASS:AMASS_XT30U-F_1x02_P5.0mm_Vertical -> RascalHat:XT30U-F-Horizontal; moved to B.Cu
- J8: footprint RascalHat:XT60-M -> RascalHat:XT60-M-Horizontal
- J9: moved to B.Cu
- moved J16 183.6 mm to (20.4, 48.1), turned to 180 degrees
- moved J15 137.4 mm to (67.7, 37.6), turned to 270 degrees
- moved J14 131.3 mm to (72.6, 37.6), turned to 270 degrees
- moved J10 126.0 mm to (2.29, 18.5), turned to 90 degrees
- moved J4 100.3 mm to (15.5, 43.2), turned to 180 degrees
- moved J12 95.7 mm to (50.8, 15.6), turned to 270 degrees
- moved J1 94.0 mm to (82.9, 23.4)
- moved J18 88.7 mm to (62.1, 24.9), turned to 90 degrees
- moved J11 79.3 mm to (45.0, 15.4), turned to 180 degrees
- moved J13 62.7 mm to (72.6, 3.43), turned to 270 degrees
- moved J8 38.5 mm to (22.1, 14.4), turned to 180 degrees
- moved J2 37.5 mm to (-28.3, 23.1), turned to 0 degrees
- moved J5 36.6 mm to (67.7, 3.43), turned to 270 degrees
- moved PWR1 35.5 mm to (14.0, 29.6), turned to 90 degrees
- moved J6 33.2 mm to (37.9, 9.20), turned to 180 degrees
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Connections:
- net A3 renamed GPIO16
- net A4 renamed GPIO19
- net A5 renamed GPIO20
- J1 pad 8: /Accelerometer MPU6050/INT -> GPIO21
- J13 pad 1: /PWM_PCA9685/P6 -> /PWM_PCA9685/P5
- J13 pad 2: /PWM_PCA9685/P7 -> /PWM_PCA9685/P6
- J13 pad 3: /PWM_PCA9685/P8 -> /PWM_PCA9685/P7
- J13 pad 4: /PWM_PCA9685/P9 -> /PWM_PCA9685/P8
- J13 pad 5: /PWM_PCA9685/P10 -> /PWM_PCA9685/P9
- J13 pad 6: /PWM_PCA9685/P11 -> /PWM_PCA9685/P10
- J13 pad 7: /PWM_PCA9685/P12 -> /PWM_PCA9685/P11
- J16 pad 2: /Radio Receiver/CH1_PWM -> /Level Shift TXB0108/B3
- J16 pad 3: /Radio Receiver/CH2_PWM -> /Level Shift TXB0108/B4
- J16 pad 4: /Radio Receiver/CH3_PWM -> /Level Shift TXB0108/B5
- J16 pad 5: /Radio Receiver/CH4_PWM -> /Level Shift TXB0108/B6
- J4 pad 1: GND -> +5V
- J4 pad 2: B8 -> B7
- J4 pad 3: B7 -> B8
- J4 pad 4: B6 -> GND
- J5 pad 1: /PWM_PCA9685/P5 -> GND
- J5 pad 2: /PWM_PCA9685/P4 -> +5V
- J5 pad 3: /PWM_PCA9685/P3 -> /PWM_PCA9685/P0
- J5 pad 4: /PWM_PCA9685/P2 -> /PWM_PCA9685/P1
- J5 pad 5: /PWM_PCA9685/P1 -> /PWM_PCA9685/P2
- J5 pad 6: /PWM_PCA9685/P0 -> /PWM_PCA9685/P3
- J5 pad 7: +5V -> /PWM_PCA9685/P4
- R1 pad 40: A6 -> GPIO21
Other:
- board size 65 x 56 mm -> 75 x 56 mm
- net class Default: clearance 0.2 -> 0.15; trace_width 0.25 -> 0.15; via_dia 0.8 -> 0.45; via_drill 0.4 -> 0.3
- rule trace_clearance: 0.2 -> 0.15
- rule trace_min: 0.2 -> 0.15
