File: FadecandyHat/FadecandyHatV1.0/FadecandyHatV1.0.sch (KiCad schematic (older format))
At the start: 17 parts, among them J1 Conn_01x03_Male, J10 Conn_01x03_Male, J11 Conn_02x08_Odd_Even, J2 Conn_01x02_Male, J3 Conn_01x03_Male, J4 Conn_01x02_Female, J5 Conn_01x03_Male, J6 Conn_01x03_Male, J7 Conn_01x03_Male, J8 Conn_01x03_Male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

Commit message: schematic updated
Connections:
- net GND: no longer H1.1, H2.1, H3.1, H4.1
- no-connect marks 0 -> 6
Changed lines of the file:
@@
-$EndComp
-$Comp
-L power:GND #PWR0102
-U 1 1 61796CD0
-P 2600 5450
-F 0 "#PWR0102" H 2600 5200 50  0001 C CNN
-F 1 "GND" H 2605 5277 50  0000 C CNN
-F 2 "" H 2600 5450 50  0001 C CNN
-F 3 "" H 2600 5450 50  0001 C CNN
-	1    2600 5450
-	1    0    0    -1
 $EndComp
 $Comp
@@
 F 3 "~" H 2600 5350 50  0001 C CNN
 	1    2600 5350
-	1    0    0    -1
-$EndComp
-$Comp
-L power:GND #PWR0103
-U 1 1 61796CC4
-P 2600 5000
-F 0 "#PWR0103" H 2600 4750 50  0001 C CNN
-F 1 "GND" H 2605 4827 50  0000 C CNN
-F 2 "" H 2600 5000 50  0001 C CNN
-F 3 "" H 2600 5000 50  0001 C CNN
-	1    2600 5000
 	1    0    0    -1
 $EndComp
@@
 $EndComp
 $Comp
-L power:GND #PWR0104
-U 1 1 6179452E
-P 2600 4550
-F 0 "#PWR0104" H 2600 4300 50  0001 C CNN
-F 1 "GND" H 2605 4377 50  0000 C CNN
-F 2 "" H 2600 4550 50  0001 C CNN
-F 3 "" H 2600 4550 50  0001 C CNN
-	1    2600 4550
-	1    0    0    -1
-$EndComp
-$Comp
 L Mechanical:MountingHole_Pad H2
 U 1 1 61794528
@@
 F 3 "~" H 2600 4450 50  0001 C CNN
 	1    2600 4450
-	1    0    0    -1
-$EndComp
-$Comp
-L power:GND #PWR0105
-U 1 1 61792FE9
-P 2600 4100
-F 0 "#PWR0105" H 2600 3850 50  0001 C CNN
-F 1 "GND" H 2605 3927 50  0000 C CNN
-F 2 "" H 2600 4100 50  0001 C CNN
-F 3 "" H 2600 4100 50  0001 C CNN
-	1    2600 4100
 	1    0    0    -1
 $EndComp
@@
 	1    0    0    -1
 $EndComp
+NoConn ~ 2600 4100
+NoConn ~ 2600 4550
+NoConn ~ 2600 5000
+NoConn ~ 2600 5450
+NoConn ~ 3100 7050
+NoConn ~ 2450 4850
 $EndSCHEMATC
