File: Prime Mover/POWER.sch (KiCad schematic (older format))
At the start: 12 parts, among them J6 Conn_01x02_Male, J7 Conn_01x02_Female, J8 Conn_01x02_Male, J9 Conn_01x02_Male

Commit message: schematic capacitors added, pcb done, gerbers generated
Parts:
- added C10, C11, C8: 0.1uF, Capacitor_SMD:C_0805_2012Metric, symbol Device:C
- added C7, C9: 27uF 16V, Capacitor_SMD:CP_Elec_5x5.3, symbol Device:CP1
- added J3: Conn_01x02_Male, RascalHat:XT30U-M-Horizontal, symbol Connector:Conn_01x02_Male
- C5: value CP1 -> 27uF 16V; footprint Capacitor_SMD:CP_Elec_4x4.5 -> Capacitor_SMD:CP_Elec_5x5.3
- J8: footprint RascalHat:XT60-M-Horizontal -> RascalHat:XT30U-M-Horizontal
Connections:
- net +3V3: now also C8.1
- net +5V: now also C10.1, C7.1
- net +BATT: now also C11.1, C9.1, J3.2 (Pin_2)
- net GND: now also C10.2, C11.2, C7.2, C8.2, C9.2, J3.1 (Pin_1)
Other:
- note added: "3V3 DCDC"
- note added: "Aux VBatt Out"
- note removed: "5V3 DCDC"
