File: Prime Mover V1.1/POWER.sch (KiCad schematic (older format))
At the start: 18 parts, among them J3 Conn_01x02_Male, J6 Conn_01x02_Male, J7 Conn_01x02_Female, J8 Conn_01x02_Male, J9 Conn_01x02_Male

Commit message: V1.1 Manufactured
Parts:
- renumbered C9 to C?, C7 to C?, C5 to C?, J7 to J?, J6 to J?, J9 to J?, J3 to J?, J8 to J?, PWR1 to PWR?, R8 to R?, R9 to R?, R10 to R?
Changed lines of the file:
@@
 XT60
 $Comp
-L Connector:Conn_01x02_Female J7
+L Connector:Conn_01x02_Female J?
 U 1 1 619F1994
 P 5350 3750
-F 0 "J7" H 5378 3726 50  0000 L CNN
+F 0 "J?" H 5378 3726 50  0000 L CNN
 F 1 "Conn_01x02_Female" H 5378 3635 50  0000 L CNN
 F 2 "RascalHat:XT30U-F-Horizontal" H 5350 3750 50  0001 C CNN
@@
 $EndComp
 $Comp
-L Connector:Conn_01x02_Male J6
+L Connector:Conn_01x02_Male J?
 U 1 1 619F2E9C
 P 5350 3300
-F 0 "J6" H 5322 3182 50  0000 R CNN
+F 0 "J?" H 5322 3182 50  0000 R CNN
 F 1 "Conn_01x02_Male" H 5322 3273 50  0000 R CNN
 F 2 "RascalHat:XT30U-M-Horizontal" H 5350 3300 50  0001 C CNN
@@
 3V3 DCDC
 $Comp
-L Rascal_KiCAD_LIB:MP1584_3V3Module PWR1
+L Rascal_KiCAD_LIB:MP1584_3V3Module PWR?
 U 1 1 61A0529B
 P 3200 3450
-F 0 "PWR1" H 3200 3085 50  0000 C CNN
+F 0 "PWR?" H 3200 3085 50  0000 C CNN
 F 1 "MP1584_3V3Module" H 3200 3176 50  0000 C CNN
 F 2 "RascalHat:MP1584-Jacobs-Parts-Module" H 3200 3750 50  0001 C CNN
@@
 $EndComp
 $Comp
-L power:+3V3 #PWR065
+L power:+3V3 #PWR?
 U 1 1 61A07296
 P 3650 3250
-F 0 "#PWR065" H 3650 3100 50  0001 C CNN
+F 0 "#PWR?" H 3650 3100 50  0001 C CNN
 F 1 "+3V3" H 3665 3423 50  0000 C CNN
 F 2 "" H 3650 3250 50  0001 C CNN
@@
 $EndComp
 $Comp
-L Device:R R8
+L Device:R R?
 U 1 1 61D39980
 P 3350 1450
-F 0 "R8" H 3420 1496 50  0000 L CNN
+F 0 "R?" H 3420 1496 50  0000 L CNN
 F 1 "470" H 3420 1405 50  0000 L CNN
 F 2 "Resistor_SMD:R_0805_2012Metric" V 3280 1450 50  0001 C CNN
@@
 $EndComp
 $Comp
-L power:+3V3 #PWR0108
+L power:+3V3 #PWR?
 U 1 1 61D39D1E
 P 3350 1200
-F 0 "#PWR0108" H 3350 1050 50  0001 C CNN
+F 0 "#PWR?" H 3350 1050 50  0001 C CNN
 F 1 "+3V3" H 3365 1373 50  0000 C CNN
 F 2 "" H 3350 1200 50  0001 C CNN
@@
 $EndComp
 $Comp
-L Device:R R9
+L Device:R R?
 U 1 1 61D3F57A
 P 3750 1450
-F 0 "R9" H 3820 1496 50  0000 L CNN
+F 0 "R?" H 3820 1496 50  0000 L CNN
 F 1 "2k2" H 3820 1405 50  0000 L CNN
 F 2 "Resistor_SMD:R_0805_2012Metric" V 3680 1450 50  0001 C CNN
@@
 $EndComp
 $Comp
-L Device:R R10
+L Device:R R?
 U 1 1 61D42780
 P 4150 1450
-F 0 "R10" H 4220 1496 50  0000 L CNN
+F 0 "R?" H 4220 1496 50  0000 L CNN
 F 1 "3k3" H 4220 1405 50  0000 L CNN
 F 2 "Resistor_SMD:R_0805_2012Metric" V 4080 1450 50  0001 C CNN
@@
 $EndComp
 $Comp
-L power:+3V3 #PWR0114
+L power:+3V3 #PWR?
 U 1 1 61D45B95
 P 4100 3350
-F 0 "#PWR0114" H 4100 3200 50  0001 C CNN
+F 0 "#PWR?" H 4100 3200 50  0001 C CNN
 F 1 "+3V3" H 4115 3523 50  0000 C CNN
 F 2 "" H 4100 3350 50  0001 C CNN
@@
 	4100 3850 4100 3750
 $Comp
-L Connector:Conn_01x02_Male J9
+L Connector:Conn_01x02_Male J?
 U 1 1 619F7430
 P 6900 3850
-F 0 "J9" H 6872 3732 50  0000 R CNN
+F 0 "J?" H 6872 3732 50  0000 R CNN
 F 1 "Conn_01x02_Male" H 6872 3823 50  0000 R CNN
 F 2 "RascalHat:XT60-M" H 6900 3850 50  0001 C CNN
@@
 $EndComp
 $Comp
-L Connector:Conn_01x02_Male J3
+L Connector:Conn_01x02_Male J?
 U 1 1 61EEA31C
 P 6700 3300
-F 0 "J3" H 6672 3182 50  0000 R CNN
+F 0 "J?" H 6672 3182 50  0000 R CNN
 F 1 "Conn_01x02_Male" H 6672 3273 50  0000 R CNN
 F 2 "RascalHat:XT30U-M-Horizontal" H 6700 3300 50  0001 C CNN
@@
 $EndComp
 $Comp
-L Connector:Conn_01x02_Male J8
+L Connector:Conn_01x02_Male J?
 U 1 1 61EEE45A
 P 8100 3300
-F 0 "J8" H 8072 3182 50  0000 R CNN
+F 0 "J?" H 8072 3182 50  0000 R CNN
 F 1 "Conn_01x02_Male" H 8072 3273 50  0000 R CNN
 F 2 "RascalHat:XT30U-M-Horizontal" H 8100 3300 50  0001 C CNN
@@
 $EndComp
 $Comp
-L Device:CP1 C9
+L Device:CP1 C?
 U 1 1 62009597
 P 8000 4050
-F 0 "C9" H 8115 4096 50  0000 L CNN
+F 0 "C?" H 8115 4096 50  0000 L CNN
 F 1 "27uF 16V" H 8115 4005 50  0000 L CNN
 F 2 "Capacitor_SMD:CP_Elec_5x5.3" H 8000 4050 50  0001 C CNN
@@
 	8000 4300 8000 4200
 $Comp
-L Device:CP1 C7
+L Device:CP1 C?
 U 1 1 6201548F
 P 4550 3600
-F 0 "C7" H 4665 3646 50  0000 L CNN
+F 0 "C?" H 4665 3646 50  0000 L CNN
 F 1 "27uF 16V" H 4665 3555 50  0000 L CNN
 F 2 "Capacitor_SMD:CP_Elec_5x5.3" H 4550 3600 50  0001 C CNN
@@
 $EndComp
 $Comp
-L Device:CP1 C5
+L Device:CP1 C?
 U 1 1 620171BC
 P 4100 3600
-F 0 "C5" H 4215 3646 50  0000 L CNN
+F 0 "C?" H 4215 3646 50  0000 L CNN
 F 1 "27uF 16V" H 4215 3555 50  0000 L CNN
 F 2 "Capacitor_SMD:CP_Elec_5x5.3" H 4100 3600 50  0001 C CNN
@@
 $EndComp
 $Comp
-L power:+3V3 #PWR072
+L power:+3V3 #PWR?
 U 1 1 62019B59
 P 5150 2100
-F 0 "#PWR072" H 5150 1950 50  0001 C CNN
+F 0 "#PWR?" H 5150 1950 50  0001 C CNN
 F 1 "+3V3" H 5165 2273 50  0000 C CNN
 F 2 "" H 5150 2100 50  0001 C CNN
