File: Prime Mover V1.1/RascalHat.kicad_pcb (KiCad board)
At the start: 2 copper layers, 75 x 56 mm, 55 parts, among them J1 Conn_01x08_Male, J10 Conn_01x04_Male, J11 Conn_01x03_Male, J12 Conn_01x03_Male, J13 Conn_01x07_Male, J14 Conn_01x07_Male, J15 Conn_01x07_Male, J16 Conn_01x06_Male, J17 Conn_01x02_Male, J18 Conn_01x07_Male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

Commit message: V1.1 Manufactured
Routing:
- net +BATT: track 114.6 -> 111.4 mm
Changed lines of the file:
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@@
     (thickness 1.6)
     (drawings 31)
-    (tracks 2083)
+    (tracks 2079)
     (zones 0)
     (modules 55)
@@
   )
   (setup
-    (last_trace_width 0.5)
+    (last_trace_width 0.15)
     (user_trace_width 0.5)
     (user_trace_width 1)
@@
   (segment (start 12.47711 35.489947) (end 13.597196 36.610033) (width 0.15) (layer B.Cu) (net 15))
   (segment (start 8.269947 35.489947) (end 12.47711 35.489947) (width 0.15) (layer B.Cu) (net 15))
-  (via (at 3.080107 35.908893) (size 0.6) (drill 0.3) (layers F.Cu B.Cu) (net 16))
   (segment (start 2.794 22.152) (end 2.669 22.152) (width 0.15) (layer B.Cu) (net 15))
   (segment (start 3.383001 32.963001) (end 3.383001 32.633445) (width 0.15) (layer B.Cu) (net 15))
@@
   (segment (start 47.525001 51.723557) (end 47.32998 51.528537) (width 0.15) (layer F.Cu) (net 15))
   (segment (start 46.45 54.69) (end 47.525001 53.614999) (width 0.15) (layer F.Cu) (net 15))
+  (via (at 3.080107 35.908893) (size 0.6) (drill 0.3) (layers F.Cu B.Cu) (net 16))
   (segment (start 3.080107 35.908893) (end 3.080107 46.219665) (width 0.15) (layer F.Cu) (net 16))
   (segment (start 2.794 19.652) (end 2.669 19.652) (width 0.15) (layer B.Cu) (net 16))
@@
   (segment (start 2.286 35.433) (end 2.286 45.849837) (width 0.15) (layer F.Cu) (net 17))
   (segment (start 2.286 45.849837) (end 7.501196 51.065033) (width 0.15) (layer F.Cu) (net 17))
-  (via (at 7.48 23.84) (size 0.6) (drill 0.3) (layers F.Cu B.Cu) (net 18))
   (segment (start 2.919 17.152) (end 2.794 17.152) (width 0.15) (layer F.Cu) (net 17))
   (segment (start 2.519 17.652) (end 2.794 17.652) (width 0.15) (layer B.Cu) (net 17))
@@
   (segment (start 12.954269 51.060009) (end 24.256164 51.060009) (width 0.15) (layer B.Cu) (net 17))
   (segment (start 11.995731 51.770009) (end 12.244269 51.770009) (width 0.15) (layer B.Cu) (net 17))
+  (via (at 7.48 23.84) (size 0.6) (drill 0.3) (layers F.Cu B.Cu) (net 18))
   (via (at 38.876273 47.247308) (size 0.6) (drill 0.3) (layers F.Cu B.Cu) (net 18))
   (segment (start 38.83 52.15) (end 38.83 47.293581) (width 0.15) (layer F.Cu) (net 18))
@@
   (segment (start 52.070097 15.350011) (end 54.030011 15.350011) (width 1) (layer F.Cu) (net 30))
   (segment (start 54.030011 15.350011) (end 56.879903 15.350011) (width 1) (layer F.Cu) (net 30))
-  (segment (start 54.030011 17.309989) (end 54.030011 15.350011) (width 0.15) (layer F.Cu) (net 30))
-  (segment (start 52.917381 17.439988) (end 53.900012 17.439988) (width 0.15) (layer F.Cu) (net 30))
-  (segment (start 52.799922 17.557447) (end 52.917381 17.439988) (width 0.15) (layer F.Cu) (net 30))
-  (segment (start 53.900012 17.439988) (end 54.030011 17.309989) (width 0.15) (layer F.Cu) (net 30))
   (via (at 55.663716 43.168007) (size 0.6) (drill 0.3) (layers F.Cu B.Cu) (net 30))
   (segment (start 56.255209 43.7595) (end 55.963715 43.468006) (width 0.15) (layer F.Cu) (net 30))
@@
     (connect_pads (clearance 0.15))
     (min_thickness 0.15)
-    (fill yes (arc_segments 32) (thermal_gap 0.5) (thermal_bridge_width 0.5))
+    (fill (arc_segments 32) (thermal_gap 0.5) (thermal_bridge_width 0.5))
     (polygon
       (pts
@@
   )
   (zone (net 1) (net_name GND) (layer B.Cu) (hatch edge 0.508)
-    (connect_pads yes (clearance 0.15))
+    (connect_pads (clearance 0.15))
     (min_thickness 0.15)
-    (fill yes (arc_segments 32) (thermal_gap 0.5) (thermal_bridge_width 0.5))
+    (fill (arc_segments 32) (thermal_gap 0.5) (thermal_bridge_width 0.5))
     (polygon
       (pts
