File: Prime Mover V1.1/RascalHat.sch (KiCad schematic (older format))
At the start: 28 parts, among them J10 Conn_01x04_Male, J11 Conn_01x03_Male, J12 Conn_01x03_Male, J13 Conn_01x07_Male, J17 Conn_01x02_Male, J2 Conn_01x09_Male, J4 Conn_01x04_Male, J5 Conn_01x07_Male

Commit message: V1.1 Manufactured
Other:
- note added: "Change 3V3 dcdc footprint!!!"
Changed lines of the file:
@@
 	1    0    0    -1
 $EndComp
+Text Notes 10600 4100 0    50   ~ 0
+Change 3V3 dcdc footprint!!!
 $EndSCHEMATC
