File: Prime Mover V1.2/Prime Mover.kicad_pcb (KiCad board)
At the start: 2 copper layers, 75 x 56 mm, 43 parts, among them IC1 MAX20404AFOC_VY+, IC2 NTS0308EPWJ, J1 Conn_01x08_Male, J10 Conn_01x04_Male, J11 Conn_01x03_Male, J12 Conn_01x03_Male, J13 Conn_01x07_Male, J14 Conn_01x07_Male, J18 Conn_01x07_Male, J2 Conn_01x09_Male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

Commit message: polished
Parts:
- added J4: Conn_01x06_Male, Connector_JST:JST_PH_B6B-PH-K_1x06_P2.00mm_Vertical, F.Cu at (12.1, 24.3)
Routing:
- net GPIO1: track 0.00 -> 48.3 mm, vias 0 -> 2
- net GPIO16: track 0.00 -> 46.7 mm, vias 0 -> 3
- net GPIO0: track 0.00 -> 45.5 mm, vias 0 -> 2
- net GND: track 452.3 -> 438.7 mm, vias 124 -> 127
- net +3V3: track 178.0 -> 187.9 mm, vias 7 -> 8
- net ENC_OUT: track 28.8 -> 32.7 mm
- net DIR: track 21.7 -> 24.6 mm
- net I2C_SDA: track 98.0 -> 99.3 mm
- net I2C_SCL: track 94.4 -> 93.1 mm
- net GPS_PWR: track 66.6 -> 67.3 mm
Other:
- board text added: "3V3 GPIO"
- board text added: "6-12V"
- board text added: "ADC"
- board text added: "Line"
- board text added: "PWM"
- board text removed: "Line Tracker"
