File: Prime Mover V1.5/Prime Mover.kicad_pcb (KiCad board)
At the start: 2 copper layers, 75 x 56 mm, 48 parts, among them IC1 NTS0308EPWJ, IC2 MAX20404AFOC_VY+, J1 Conn_01x06_Male, J10 Conn_01x07_Male, J11 Conn_01x02_Male, J12 Conn_01x08_Male, J2 Conn_01x04_Male, J3 Conn_01x03_Male, J4 Conn_01x09_Male, J5 Conn_01x03_Male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

Commit message: PCBA quoted - generated BOM & POS
Changed lines of the file:
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@@
       (drillshape 0)
       (scaleselection 1)
-      (outputdirectory "Prime Mover V1.4 Gerbers/")
+      (outputdirectory "Prime Mover V1.5 POS/")
     )
   )
@@
     (fp_line (start -1 -0.625) (end 1 -0.625) (layer "F.Fab") (width 0.1))
     (fp_line (start 1 0.625) (end -1 0.625) (layer "F.Fab") (width 0.1))
-    (pad "1" smd roundrect (at -0.9125 0 90) (size 1.025 1.4) (layers "F.Cu" "F.Paste" "F.Mask") (roundrect_rratio 0.243902)
+    (pad "1" smd roundrect (at -0.9125 0 90) (size 1.025 1.4) (layers "F.Cu" "F.Paste" "F.Mask") (roundrect_rratio 0.243902439)
       (net 1 "GND") (pintype "passive"))
-    (pad "2" smd roundrect (at 0.9125 0 90) (size 1.025 1.4) (layers "F.Cu" "F.Paste" "F.Mask") (roundrect_rratio 0.243902)
+    (pad "2" smd roundrect (at 0.9125 0 90) (size 1.025 1.4) (layers "F.Cu" "F.Paste" "F.Mask") (roundrect_rratio 0.243902439)
       (net 107 "Net-(D2-Pad1)") (pintype "passive"))
     (model "${KICAD6_3DMODEL_DIR}/Resistor_SMD.3dshapes/R_0805_2012Metric.wrl"
@@
     (fp_line (start 1 0.625) (end -1 0.625) (layer "F.Fab") (width 0.1))
     (fp_line (start 1 -0.625) (end 1 0.625) (layer "F.Fab") (width 0.1))
-    (pad "1" smd roundrect (at -0.9125 0 90) (size 1.025 1.4) (layers "F.Cu" "F.Paste" "F.Mask") (roundrect_rratio 0.243902)
+    (pad "1" smd roundrect (at -0.9125 0 90) (size 1.025 1.4) (layers "F.Cu" "F.Paste" "F.Mask") (roundrect_rratio 0.243902439)
       (net 1 "GND") (pintype "passive"))
-    (pad "2" smd roundrect (at 0.9125 0 90) (size 1.025 1.4) (layers "F.Cu" "F.Paste" "F.Mask") (roundrect_rratio 0.243902)
+    (pad "2" smd roundrect (at 0.9125 0 90) (size 1.025 1.4) (layers "F.Cu" "F.Paste" "F.Mask") (roundrect_rratio 0.243902439)
       (net 109 "Net-(D4-Pad1)") (pintype "passive"))
     (model "${KICAD6_3DMODEL_DIR}/Resistor_SMD.3dshapes/R_0805_2012Metric.wrl"
@@
     (fp_line (start -1 -0.625) (end 1 -0.625) (layer "F.Fab") (width 0.1))
     (fp_line (start 1 0.625) (end -1 0.625) (layer "F.Fab") (width 0.1))
-    (pad "1" smd roundrect (at -0.9125 0 90) (size 1.025 1.4) (layers "F.Cu" "F.Paste" "F.Mask") (roundrect_rratio 0.243902)
+    (pad "1" smd roundrect (at -0.9125 0 90) (size 1.025 1.4) (layers "F.Cu" "F.Paste" "F.Mask") (roundrect_rratio 0.243902439)
       (net 1 "GND") (pintype "passive"))
-    (pad "2" smd roundrect (at 0.9125 0 90) (size 1.025 1.4) (layers "F.Cu" "F.Paste" "F.Mask") (roundrect_rratio 0.243902)
+    (pad "2" smd roundrect (at 0.9125 0 90) (size 1.025 1.4) (layers "F.Cu" "F.Paste" "F.Mask") (roundrect_rratio 0.243902439)
       (net 108 "Net-(D3-Pad1)") (pintype "passive"))
     (model "${KICAD6_3DMODEL_DIR}/Resistor_SMD.3dshapes/R_0805_2012Metric.wrl"
@@
   (gr_circle (center 29.51 15.62) (end 30.93 16.04) (layer "Edge.Cuts") (width 0.05) (fill none))
   (gr_arc (start -1.475 -7) (mid -3.975 -4.5) (end -6.475 -7) (layer "Edge.Cuts") (width 0.05))
-  (gr_arc (start 22.97 -4.35) (mid 23.262893 -5.057106) (end 23.97 -5.35) (layer "Edge.Cuts") (width 0.05))
+  (gr_arc (start 22.97 -4.35) (mid 23.262894 -5.057106) (end 23.97 -5.35) (layer "Edge.Cuts") (width 0.05))
   (gr_arc (start -19.5 28) (mid -21.62132 27.12132) (end -22.5 25) (layer "Edge.Cuts") (width 0.05))
-  (gr_arc (start 17 14.25) (mid 17.292893 13.542894) (end 18 13.25) (layer "Edge.Cuts") (width 0.05))
-  (gr_arc (start 47.95 3.23) (mid 47.657107 3.937106) (end 46.95 4.23) (layer "Edge.Cuts") (width 0.05))
+  (gr_arc (start 17 14.25) (mid 17.292894 13.542894) (end 18 13.25) (layer "Edge.Cuts") (width 0.05))
+  (gr_arc (start 47.95 3.23) (mid 47.657106 3.937106) (end 46.95 4.23) (layer "Edge.Cuts") (width 0.05))
   (gr_line (start -7.475 -28) (end -19.5 -28) (layer "Edge.Cuts") (width 0.05))
   (gr_line (start 52.5 25) (end 52.5 18.12) (layer "Edge.Cuts") (width 0.05))
@@
     (connect_pads (clearance 0.15))
     (min_thickness 0.15) (filled_areas_thickness no)
-    (fill yes (thermal_gap 0.508) (thermal_bridge_width 0.508))
+    (fill (thermal_gap 0.508) (thermal_bridge_width 0.508))
     (polygon
       (pts
