File: Prime Mover V1.6/POWER.kicad_sch (KiCad schematic)
At the start: 15 parts, among them IC2 MAX20404AFOC_VY+, J11 Conn_01x02_Male

Commit message: PCBA quoted - generated BOM & POS
Parts:
- C10, C9: value 1.0uF -> 1.0uF 16v
- C2: value 0.1uF -> 0.1uF 16v
- C3: value 2.2uF -> 2.2uF 10v
- C4, C6, C8: value 22uF -> 22uF 10v
- C5, C7: value 4.7uF -> 4.7uF 16v
- R6: value R -> 120k
- R7: value R -> 22k
Other:
- note added: "115.5k=22k*(5V/0.8V-1)"
- note added: "R6=R7*(Vout/0.8V-1)"
- note added: "Vout=0.8V(R6/R7+1)"
Changed lines of the file:
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@@
     (stroke (width 0) (type default) (color 0 0 0 0))
+  )
+  (text "Vout=0.8V(R6/R7+1)" (at 152.4 71.12 0)
+    (effects (font (size 1.27 1.27)) (justify left bottom))
   )
   (text "For setting Vout" (at 133.35 74.93 0)
@@
     (effects (font (size 1.27 1.27)) (justify left bottom))
   )
+  (text "R6=R7*(Vout/0.8V-1)" (at 152.4 68.58 0)
+    (effects (font (size 1.27 1.27)) (justify left bottom))
+  )
+  (text "115.5k=22k*(5V/0.8V-1)" (at 175.26 68.58 0)
+    (effects (font (size 1.27 1.27)) (justify left bottom))
+  )
   (global_label "LX" (shape input) (at 92.71 92.71 180) (fields_autoplaced)
     (effects (font (size 1.27 1.27)) (justify right))
@@
       (effects (font (size 1.27 1.27)) (justify left))
     )
-    (property "Value" "22uF" (id 1) (at 179.451 119.9766 0)
+    (property "Value" "22uF 10v" (id 1) (at 179.451 119.9766 0)
       (effects (font (size 1.27 1.27)) (justify left))
     )
@@
       (effects (font (size 1.27 1.27)) (justify left))
     )
-    (property "Value" "1.0uF" (id 1) (at 221.361 97.1166 0)
+    (property "Value" "1.0uF 16v" (id 1) (at 221.361 97.1166 0)
       (effects (font (size 1.27 1.27)) (justify left))
     )
@@
       (effects (font (size 1.27 1.27)) (justify left))
     )
-    (property "Value" "22uF" (id 1) (at 201.041 119.9766 0)
+    (property "Value" "22uF 10v" (id 1) (at 201.041 119.9766 0)
       (effects (font (size 1.27 1.27)) (justify left))
     )
@@
       (effects (font (size 1.27 1.27)) (justify left))
     )
-    (property "Value" "0.1uF" (id 1) (at 142.621 122.5166 0)
+    (property "Value" "0.1uF 16v" (id 1) (at 142.621 122.5166 0)
       (effects (font (size 1.27 1.27)) (justify left))
     )
@@
       (effects (font (size 1.27 1.27)) (justify left))
     )
-    (property "Value" "22uF" (id 1) (at 189.611 119.9766 0)
+    (property "Value" "22uF 10v" (id 1) (at 189.611 119.9766 0)
       (effects (font (size 1.27 1.27)) (justify left))
     )
@@
       (effects (font (size 1.27 1.27)) (justify left))
     )
-    (property "Value" "R" (id 1) (at 152.908 89.4966 0)
+    (property "Value" "22k" (id 1) (at 152.908 89.4966 0)
       (effects (font (size 1.27 1.27)) (justify left))
     )
@@
       (effects (font (size 1.27 1.27)) (justify left))
     )
-    (property "Value" "4.7uF" (id 1) (at 198.501 97.1166 0)
+    (property "Value" "4.7uF 16v" (id 1) (at 198.501 97.1166 0)
       (effects (font (size 1.27 1.27)) (justify left))
     )
@@
       (effects (font (size 1.27 1.27)) (justify left))
     )
-    (property "Value" "1.0uF" (id 1) (at 209.931 97.1166 0)
+    (property "Value" "1.0uF 16v" (id 1) (at 209.931 97.1166 0)
       (effects (font (size 1.27 1.27)) (justify left))
     )
@@
       (effects (font (size 1.27 1.27)) (justify left))
     )
-    (property "Value" "4.7uF" (id 1) (at 187.071 97.1166 0)
+    (property "Value" "4.7uF 16v" (id 1) (at 187.071 97.1166 0)
       (effects (font (size 1.27 1.27)) (justify left))
     )
@@
       (effects (font (size 1.27 1.27)) (justify left))
     )
-    (property "Value" "R" (id 1) (at 152.908 79.3366 0)
+    (property "Value" "120k" (id 1) (at 152.908 79.3366 0)
       (effects (font (size 1.27 1.27)) (justify left))
     )
@@
       (effects (font (size 1.27 1.27)) (justify left))
     )
-    (property "Value" "2.2uF" (id 1) (at 169.291 97.1166 0)
-      (effects (font (size 1.27 1.27)) (justify left))
-    )
+    (property "Value" "2.2uF 10v" (id 1) (at 169.291 97.1166 0)
+      (effects (font (size 1.27 1.27)) (justify left))
+    )
