File: Prime Mover V1.6/_autosave-Prime Mover.kicad_pcb (KiCad board)
At the start: 2 copper layers, 75 x 56 mm, 48 parts, among them IC1 NTS0308EPWJ, IC2 MAX20404AFOC_VY+, J1 Conn_01x06_Male, J10 Conn_01x07_Male, J11 Conn_01x02_Male, J12 Conn_01x08_Male, J2 Conn_01x04_Male, J3 Conn_01x03_Male, J4 Conn_01x09_Male, J5 Conn_01x03_Male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

Commit message: PCBA quoted - generated BOM & POS
Parts:
- C1: value 0.1uF -> 0.1uF 16V
- C10, C9: value 1.0uF -> 1.0uF 16v
- C2: value 0.1uF -> 0.1uF 16v
- C3: value 2.2uF -> 2.2uF 10v
- C4, C6, C8: value 22uF -> 22uF 10v
- C5, C7: value 4.7uF -> 4.7uF 16v
- R6: value R -> 120k
- R7: value R -> 22k
Routing:
- net +BATT: track 134.9 -> 149.0 mm
- net GND: track 485.8 -> 491.7 mm
- net LX: track 11.0 -> 11.6 mm
Other:
- board text added: "Prime Mover V1.6"
- board text removed: "Prime Mover V1.5"
